File: hardware/To-mate-Oh.brd (EAGLE design)
At the start: 22.2 x 33.8 mm, 25 parts, among them IC1 Tiny45-20-SMT

Commit message: Added readme
Update README.md

Update README.md

Update README.md

Update README.md

Update README.md

Minor cosmetics

Minor cosmetics

Minor cosmetics

Update README.md
Parts:
- BAT: value (none) -> 3.3-5.0V
- C1: value 100uF -> 1-10uF
- JP1: value (none) -> JGND1
- JP2: value (none) -> JGND2
- JP3: value (none) -> JPB1
- JP4: value (none) -> JPB2
- JP5: value (none) -> JVCC1
- JP6: value (none) -> JVCC2
- LED1, LED2, LED3, LED5, LED6: value (none) -> Blue
- renumbered LED4 to STATUS, U$1 to CAP_SENSE
Connections:
- net VBAT renamed BAT+
Routing:
- net PB4: track 30.2 -> 27.4 mm
Other:
- board text added: "To-mate-Oh board, v.1.1 Copyright © 2014 con-f-use Use permitted under GNU General Public License v3.0 or later. To-mate-Oh is based on POMODORO by FakuFaku. Disconnect battery and supply your own voltage to program."
- board text removed: "To-mate-Oh board, v.1.1 Copyright © 2014 con-f-use Use permitted under GNU General Public License v3.0 or later. To-mate-Oh is based on POMODORO by FakuFaku"
